Commit message: Complete Assignment 6 MoveIt configuration package setup

File: bulls_bot/urdf/bulls.urdf (robot description, URDF)
Before this commit: robot bulls_bot, 1 links, 0 joints
Links:
- added link gripper_base; collision box size=0.2 0.04 0.04; visual box size=0.2 0.04 0.04
- added link left_finger; collision box size=0.02 0.03 0.08; visual box size=0.02 0.03 0.08
- added link link_1; collision cylinder length=0.4 radius=0.08; visual cylinder length=0.4 radius=0.08
- added link link_2; collision cylinder length=0.4 radius=0.06; visual cylinder length=0.4 radius=0.06
- added link link_3; collision cylinder length=0.3 radius=0.05; visual cylinder length=0.3 radius=0.05
- added link right_finger; collision box size=0.02 0.03 0.08; visual box size=0.02 0.03 0.08
- link base_link: geometry collision cylinder length=0.6 radius=0.2; visual cylinder length=0.6 radius=0.2
Joints:
- added joint arm_0_joint: type revolute, parent base_link, child link_1, origin xyz=0 0 0.6 rpy=0 0 0, axis 0 0 1, limit lower=-3.1416 upper=3.1416 effort=10.0 velocity=1.0
- added joint arm_1_joint: type revolute, parent link_1, child link_2, origin xyz=0 0 0.4 rpy=0 0 0, axis 0 1 0, limit lower=-1.5708 upper=1.5708 effort=10.0 velocity=1.0
- added joint arm_2_joint: type revolute, parent link_2, child link_3, origin xyz=0 0 0.4 rpy=0 0 0, axis 0 1 0, limit lower=-2.0 upper=2.0 effort=10.0 velocity=1.0
- added joint gripper_base_joint: type fixed, parent link_3, child gripper_base, origin xyz=0 0 0.3 rpy=0 0 0
- added joint gripper_finger_joint_1: type prismatic, parent gripper_base, child left_finger, origin xyz=-0.08 0 0.04 rpy=0 0 0, axis 1 0 0, limit lower=0.0 upper=0.06 effort=5.0 velocity=0.5
- added joint gripper_finger_joint_2: type prismatic, parent gripper_base, child right_finger, origin xyz=0.08 0 0.04 rpy=0 0 0, axis -1 0 0, limit lower=0.0 upper=0.06 effort=5.0 velocity=0.5
